Commit message: Publish exact Onshape wrist URDF viewer

File: models/urdf/ruggedized-wrist.urdf (robot description, URDF)
Before this commit: robot ruggedized_wrist_web, 6 links, 5 joints
Links:
- removed link linear_probe
- removed link pitch_drive
- removed link probe_roll_output
- removed link wrist_mount
- removed link wrist_pitch_link
- added link mount_to_arm; visual mesh filename=meshes/mount-to-arm.glb
- added link pitch_motor; visual mesh filename=meshes/pitch-motor.glb
- added link pitch_pulley; visual mesh filename=meshes/pitch-pulley.glb
- added link pitch_pulley_connector; visual mesh filename=meshes/pitch-pulley-connector.glb
- added link roll_motor_bracket; visual mesh filename=meshes/roll-motor-bracket.glb
- added link roll_motor_housing; visual mesh filename=meshes/roll-motor-housing.glb
- added link roll_output; visual mesh filename=meshes/roll-output.glb
- added link root
- link wrist_base: geometry visual mesh filename=meshes/base.glb
Joints:
- removed joint base_to_pitch_drive
- removed joint roll_output_to_probe
- added joint base_to_pitch_motor: type fixed, parent wrist_base, child pitch_motor, origin xyz=0.0223882 0.0334 0.0159693
- added joint bracket_to_roll_motor: type fixed, parent roll_motor_bracket, child roll_motor_housing, origin xyz=0.0212802 -0.0176901 -0.0208303 rpy=0 -0.0947442 0
- added joint connector_to_pulley: type fixed, parent pitch_pulley_connector, child pitch_pulley, origin xyz=0 -0.0099 0 rpy=0 -0.0947442 0
- added joint pitch_drive_fixed: type fixed, parent pitch_motor, child pitch_pulley_connector, origin xyz=-0.0223882 -0.0471 -0.0159693
- added joint root_to_base: type fixed, parent root, child wrist_base, origin xyz=0 -0.00025 0.04545
- joint base_to_mount: child wrist_mount -> mount_to_arm
- joint wrist_pitch_joint: child wrist_pitch_link -> roll_motor_bracket
- joint wrist_roll_joint: child probe_roll_output -> roll_output; origin xyz=-0.001159 -0.031650 0.012195 rpy=3.141593 -0.094744 0 -> xyz=-0.0192142 -0.0139599 0.0323; parent wrist_pitch_link -> roll_motor_housing

Commit message: Publish high-resolution J9 and Gecko fix

File: models/urdf/ruggedized-wrist.urdf (robot description, URDF)
Before this commit: robot ruggedized_wrist_onshape, 9 links, 8 joints
Links:
- added link gecko_attachment; visual mesh filename=meshes/gecko.glb scale=0.00045 0.00045 0.00045
Joints:
- added joint roll_output_to_gecko: type fixed, parent roll_output, child gecko_attachment, origin xyz=0 0 0.0087

Commit message: Publish cache-busted J9 model and application section

File: models/urdf/ruggedized-wrist.urdf (robot description, URDF)
Before this commit: robot ruggedized_wrist_onshape, 10 links, 9 joints
Links:
- link gecko_attachment: geometry visual mesh filename=meshes/gecko.glb?v=20260731-j9-gecko-2 scale=0.00045 0.00045 0.00045
- link mount_to_arm: geometry visual mesh filename=meshes/mount-to-arm.glb?v=20260731-j9-gecko-2
- link pitch_motor: geometry visual mesh filename=meshes/pitch-motor.glb?v=20260731-j9-gecko-2
- link pitch_pulley: geometry visual mesh filename=meshes/pitch-pulley.glb?v=20260731-j9-gecko-2
- link pitch_pulley_connector: geometry visual mesh filename=meshes/pitch-pulley-connector.glb?v=20260731-j9-gecko-2
- link roll_motor_bracket: geometry visual mesh filename=meshes/roll-motor-bracket.glb?v=20260731-j9-gecko-2
- link roll_motor_housing: geometry visual mesh filename=meshes/roll-motor-housing.glb?v=20260731-j9-gecko-2
- link roll_output: geometry visual mesh filename=meshes/roll-output.glb?v=20260731-j9-gecko-2
- link wrist_base: geometry visual mesh filename=meshes/base.glb?v=20260731-j9-gecko-2

Commit message: Publish sharper no-shadow CAD and Tory portrait

File: models/urdf/ruggedized-wrist.urdf (robot description, URDF)
Before this commit: robot ruggedized_wrist_onshape, 10 links, 9 joints
Links:
- link gecko_attachment: geometry visual mesh filename=meshes/gecko.glb?v=20260731-cad-clear-3 scale=0.00045 0.00045 0.00045
- link mount_to_arm: geometry visual mesh filename=meshes/mount-to-arm.glb?v=20260731-cad-clear-3
- link pitch_motor: geometry visual mesh filename=meshes/pitch-motor.glb?v=20260731-cad-clear-3
- link pitch_pulley: geometry visual mesh filename=meshes/pitch-pulley.glb?v=20260731-cad-clear-3
- link pitch_pulley_connector: geometry visual mesh filename=meshes/pitch-pulley-connector.glb?v=20260731-cad-clear-3
- link roll_motor_bracket: geometry visual mesh filename=meshes/roll-motor-bracket.glb?v=20260731-cad-clear-3
- link roll_motor_housing: geometry visual mesh filename=meshes/roll-motor-housing.glb?v=20260731-cad-clear-3
- link roll_output: geometry visual mesh filename=meshes/roll-output.glb?v=20260731-cad-clear-3
- link wrist_base: geometry visual mesh filename=meshes/base.glb?v=20260731-cad-clear-3

Commit message: Publish original STL interactive wrist

File: models/urdf/ruggedized-wrist.urdf (robot description, URDF)
Before this commit: robot ruggedized_wrist_onshape, 10 links, 9 joints
Links:
- link gecko_attachment: geometry visual mesh filename=original-stl-v1/gecko-original.stl scale=0.00045 0.00045 0.00045
- link mount_to_arm: geometry visual mesh filename=original-stl-v1/mountToArm.stl
- link pitch_motor: geometry visual mesh filename=original-stl-v1/KAA15CL0a5047.stl; visual mesh filename=original-stl-v1/_3D______5044_5600_6709_2023_10_245047.stl
- link pitch_pulley: geometry visual mesh filename=original-stl-v1/PitchMotorPulley.stl
- link pitch_pulley_connector: geometry visual mesh filename=original-stl-v1/PitchMotorPulleyConnector.stl
- link roll_motor_bracket: geometry visual mesh filename=original-stl-v1/RollMotorBracket.stl
- link roll_motor_housing: geometry visual mesh filename=original-stl-v1/_2____44380227.stl; visual mesh filename=original-stl-v1/_303740227.stl
- link roll_output: geometry visual mesh filename=original-stl-v1/______44380227.stl
- link wrist_base: geometry visual mesh filename=original-stl-v1/Base.stl
